Commit message: Added Robotiq Gripper model and mockup realsense camera box

File: install/robot_gdl_description/share/robot_gdl_description/urdf/robot_gdl.urdf.xacro (robot description, xacro)
@@ -1 +1,21 @@
-/home/javier-rojas/Documents/Doctorado/3er_Semestre/ur_pick_and_place/src/robot_gdl_description/urdf/robot_gdl.urdf.xacro
+<?xml version="1.0"?>
+<robot name="my_robot_cell" xmlns:xacro="http://ros.org/wiki/xacro">
+  <xacro:include filename="$(find robot_gdl_description)/urdf/robot_gdl_macro.xacro"/>
+  <xacro:arg name="ur_type" default="ur5e"/>
+  <xacro:arg name="joint_limits_parameters_file" default="$(find ur_description)/config/$(arg ur_type)/joint_limits.yaml"/>
+  <xacro:arg name="kinematics_parameters_file" default="$(find ur_description)/config/$(arg ur_type)/default_kinematics.yaml"/>
+  <xacro:arg name="physical_parameters_file" default="$(find ur_description)/config/$(arg ur_type)/physical_parameters.yaml"/>
+  <xacro:arg name="visual_parameters_file" default="$(find ur_description)/config/$(arg ur_type)/visual_parameters.yaml"/>
+  <link name="world"/>
+  <!--This will create the scene where the robot is located in-->
+  <xacro:robot_gdl
+    parent="world"
+    ur_type="$(arg ur_type)"
+    joint_limits_parameters_file="$(arg joint_limits_parameters_file)"
+    kinematics_parameters_file="$(arg kinematics_parameters_file)"
+    physical_parameters_file="$(arg physical_parameters_file)"
+    visual_parameters_file="$(arg visual_parameters_file)"
+    >
+      <origin xyz="0 0 1" rpy="0 0 0" />
+  </xacro:robot_gdl>
+</robot>

File: install/robot_gdl_description/share/robot_gdl_description/urdf/robot_gdl_macro.xacro (robot description, xacro)
@@ -1 +1,73 @@
-/home/javier-rojas/Documents/Doctorado/3er_Semestre/ur_pick_and_place/src/robot_gdl_description/urdf/robot_gdl_macro.xacro
+<?xml version="1.0"?>
+<robot xmlns:xacro="http://ros.org/wiki/xacro">
+  <xacro:include filename="$(find ur_description)/urdf/ur_macro.xacro"/>
+  <xacro:macro name="robot_gdl" params="
+    parent
+    *origin
+    ur_type
+    joint_limits_parameters_file
+    kinematics_parameters_file
+    physical_parameters_file
+    visual_parameters_file
+    ">
+    <link name="robot_mount"/>
+    <joint name="base_to_robot_mount" type="fixed">
+      <parent link="world"/>
+      <child link="robot_mount"/>
+      <origin xyz="0.0 0.0 0" rpy="0 0 0" />
+    </joint>
+    <!--This will create the specific robot-->
+    <xacro:ur_robot
+      name="${ur_type}"
+      tf_prefix="${ur_type}_"
+      parent="robot_mount"
+      joint_limits_parameters_file="${joint_limits_parameters_file}"
+      kinematics_parameters_file="${kinematics_parameters_file}"
+      physical_parameters_file="${physical_parameters_file}"
+      visual_parameters_file="${visual_parameters_file}"
+      generate_ros2_control_tag="false"
+    >
+      <origin xyz="0 0 0" rpy="0 0 0" />
+    </xacro:ur_robot>
+    <!-- Realsense camera link -->
+    <link name="realsense_link">
+      <visual>
+        <geometry>
+          <box size="0.05 0.02 0.02"/> <!-- Tamaño aproximado -->
+        </geometry>
+        <origin xyz="0 0 0" rpy="0 0 0"/>
+        <material name="gray">
+          <color rgba="0.5 0.5 0.5 1.0"/>
+        </material>
+      </visual>
+      <collision>
+        <geometry>
+          <box size="0.05 0.02 0.02"/>
+        </geometry>
+        <origin xyz="0 0 0" rpy="0 0 0"/>
+      </collision>
+      <inertial>
+        <mass value="0.1"/>
+        <origin xyz="0 0 0" rpy="0 0 0"/>
+        <inertia
+          ixx="1e-4" iyy="1e-4" izz="1e-4"
+          ixy="0.0" ixz="0.0" iyz="0.0"/>
+      </inertial>
+    </link>
+    <!-- Fixed joint between tool0 and camera -->
+    <joint name="tool0_to_realsense" type="fixed">
+      <parent link="${ur_type}_tool0"/>
+      <child link="realsense_link"/>
+      <!-- Ajusta la posición de la cámara respecto al efector final -->
+      <origin xyz="0.0 -0.08 -0.05" rpy="0 0 0"/>
+    </joint>
+  <!-- Robotiq 2F-85 Gripper -->
+  <xacro:include filename="$(find robotiq_description)/urdf/robotiq_2f_85_macro.urdf.xacro"/>
+  <xacro:robotiq_gripper
+    name="robotiq_85"
+    prefix=""
+    parent="${ur_type}_tool0">
+    <origin xyz="0 0 0" rpy="0 0 0"/>
+  </xacro:robotiq_gripper>
+  </xacro:macro>
+</robot>
